Commit message: Initial Commit

File: src/pomona_description/urdf/xacro/gazebo_plugins.xacro (robot description, xacro)
@@ -21,4 +21,7 @@
         <namespace>/</namespace>
       </ros>
+      <!-- Two wheels per side → must declare 2 pairs, else the plugin
+           aborts with "Inconsistent number of joints specified". -->
+      <num_wheel_pairs>2</num_wheel_pairs>
       <!-- Left side wheels (front_left + rear_left) -->
       <left_joint>front_left_wheel</left_joint>
@@ -40,18 +43,7 @@
       <update_rate>50.0</update_rate>
     </plugin>
-    <!-- Joint state publisher for arm + gripper visualisation -->
-    <plugin name="pomona_joint_states" filename="libgazebo_ros_joint_state_publisher.so">
-      <ros>
-        <remapping>~/out:=joint_states</remapping>
-      </ros>
-      <update_rate>50</update_rate>
-      <joint_name>joint1</joint_name>
-      <joint_name>joint2</joint_name>
-      <joint_name>joint3</joint_name>
-      <joint_name>joint4</joint_name>
-      <joint_name>joint5</joint_name>
-      <joint_name>joint6</joint_name>
-      <joint_name>finger_joint</joint_name>
-    </plugin>
+    <!-- NOTE: arm/gripper joint_states are published by joint_state_broadcaster
+         (ros2_control.xacro), not by libgazebo_ros_joint_state_publisher, to
+         avoid two publishers racing on /joint_states. -->
   </gazebo>
   <!-- ════════════════════════════════════════════════════════════════════

File: src/pomona_description/urdf/xacro/pomona.xacro (robot description, xacro)
@@ -21,9 +21,12 @@
   <!-- ── mobile base ──────────────────────────────────────────────────── -->
   <xacro:include filename="$(find pomona_description)/urdf/xacro/scout_v2.xacro"/>
+  <!-- ── mounting box (white cuboid carrying arm + display) ───────────── -->
+  <xacro:include filename="$(find pomona_description)/urdf/xacro/mount.xacro"/>
   <!-- ── manipulator ──────────────────────────────────────────────────── -->
   <xacro:include filename="$(find pomona_description)/urdf/xacro/xarm6.xacro"/>
   <xacro:xarm6 prefix=""/>
   <!-- Mount xArm6 on Scout base: 0.212 forward of base centre, 0.26 up
-       (from goldmines/.../scout_xarm_gripper.xacro) -->
+       (from goldmines/.../scout_xarm_gripper.xacro). The white mounting box
+       (box_link, see mount.xacro) physically fills the gap up to this point. -->
   <joint name="arm_mount_joint" type="fixed">
     <parent link="base_link"/>
@@ -42,7 +45,10 @@
   <!-- ── sensors (LiDAR, IMU, camera links) ───────────────────────────── -->
   <xacro:include filename="$(find pomona_description)/urdf/xacro/sensors.xacro"/>
-  <!-- ── Gazebo plugins (conditional) ─────────────────────────────────── -->
+  <!-- ── UVC lamp bar (front of box, below LiDAR) ─────────────────────── -->
+  <xacro:include filename="$(find pomona_description)/urdf/xacro/uvc_lamps.xacro"/>
+  <!-- ── Gazebo plugins + ros2_control (conditional) ──────────────────── -->
   <xacro:if value="${use_sim}">
     <xacro:include filename="$(find pomona_description)/urdf/xacro/gazebo_plugins.xacro"/>
+    <xacro:include filename="$(find pomona_description)/urdf/xacro/ros2_control.xacro"/>
   </xacro:if>
 </robot>

File: src/pomona_description/urdf/xacro/sensors.xacro (robot description, xacro)
@@ -12,27 +12,33 @@
 <robot xmlns:xacro="http://ros.org/wiki/xacro">
   <!-- ════════════════════════════════════════════════════════════════════
-       1. Robosense LiDAR (mounted on base_link, frame = rslidar)
-       Origin: 0 0 0.138 from base_link  (from bringup_minimal.launch)
+       1. Robosense LiDAR (frame = rslidar)
+       The real unit sits at the FRONT of the mounting box, not floating
+       above the base centre. Mounted on box_link with the original
+       laser_Link transform from scout_xarm_base (xyz 0.37655 0 0.003).
+       Visual uses the ported laser_link mesh; collision is a cheap cylinder.
        ════════════════════════════════════════════════════════════════════ -->
   <link name="rslidar">
     <visual>
       <origin xyz="0 0 0" rpy="0 0 0"/>
-      <geometry><cylinder length="0.07" radius="0.05"/></geometry>
-      <material name="dark"/>
+      <geometry>
+        <mesh filename="package://pomona_description/meshes/mount/laser_link.stl"/>
+      </geometry>
+      <material name="white"/>
     </visual>
     <collision>
-      <origin xyz="0 0 0" rpy="0 0 0"/>
-      <geometry><cylinder length="0.07" radius="0.05"/></geometry>
+      <origin xyz="0 0 0.04" rpy="0 0 0"/>
+      <geometry><cylinder length="0.09" radius="0.05"/></geometry>
     </collision>
     <inertial>
-      <mass value="0.83"/>
-      <origin xyz="0 0 0"/>
-      <xacro:cylinder_inertia m="0.83" r="0.05" h="0.07"/>
+      <origin xyz="-0.00029458 -1.102E-05 0.035775" rpy="0 0 0"/>
+      <mass value="0.58508"/>
+      <inertia ixx="0.00062907" ixy="-3.4247E-08" ixz="6.994E-08"
+               iyy="0.00063026" iyz="-4.8147E-08"  izz="0.00074925"/>
     </inertial>
   </link>
   <joint name="rslidar_joint" type="fixed">
-    <parent link="base_link"/>
+    <parent link="box_link"/>
     <child  link="rslidar"/>
-    <origin xyz="0 0 0.138" rpy="0 0 0"/>
+    <origin xyz="0.37655 0 0.003" rpy="0 0 0"/>
   </joint>
   <!-- ════════════════════════════════════════════════════════════════════
