Commit message: Split sim robot into pomona_original / pomona_uvc; fix lidar gzserver crash
   - Two self-contained description models: pomona_original (full xArm6 + AG95 +
     D435 + ros2_control) and pomona_uvc (UV-C boom, no arm/camera/control)
   - Per-model launch, state-publisher, and SDF; SDFs regenerated from xacro
   - Fix gzserver SIGSEGV after spawn: rslidar is now gpu_ray, not CPU ray
     (CPU ray's ODE raycast segfaults with no render context — pomona_uvc has
     no camera to init one)
   - Sweep docs/comments to the two-model layout; drop superseded models/pomona

File: src/pomona_description/urdf/pomona_original/xacro/gazebo_plugins.xacro (robot description, xacro)
@@ -8,5 +8,5 @@
     - libgazebo_ros_diff_drive.so       — Scout V2 skid-steer (4 wheels)
     - libgazebo_ros_joint_state_publisher.so — joint_states for arm + gripper
-    - libgazebo_ros_ray_sensor.so       — rslidar /scan + /points
+    - libgazebo_ros_ray_sensor.so       — rslidar (gpu_ray) → /scan
     - libgazebo_ros_camera.so           — D435 RGB + depth
     - libgazebo_ros_imu_sensor.so       — Xsens IMU /imu/data
@@ -31,5 +31,5 @@
       <right_joint>rear_right_wheel</right_joint>
       <wheel_separation>0.58306</wheel_separation>
-      <wheel_diameter>0.32918</wheel_diameter>
+      <wheel_diameter>${2 * wheel_radius}</wheel_diameter>
       <max_wheel_torque>50.0</max_wheel_torque>
       <max_wheel_acceleration>2.0</max_wheel_acceleration>
@@ -51,5 +51,9 @@
        ════════════════════════════════════════════════════════════════════ -->
   <gazebo reference="rslidar">
-    <sensor name="rslidar" type="ray">
+    <!-- gpu_ray (not CPU "ray"): the CPU ray path (ODEMultiRayShape) can segfault
+         in dSpaceCollide2 when gzserver has no rendering context. Here the D435
+         camera happens to provide one, but gpu_ray is the robust choice (renders
+         the scan instead of ODE-raycasting) and is faster. -->
+    <sensor name="rslidar" type="gpu_ray">
       <always_on>true</always_on>
       <visualize>true</visualize>

File: src/pomona_description/urdf/pomona_original/xacro/pomona.xacro (robot description, xacro)
@@ -18,11 +18,11 @@
   <xacro:property name="use_sim" value="$(arg use_sim)"/>
   <!-- ── shared utilities ─────────────────────────────────────────────── -->
-  <xacro:include filename="$(find pomona_description)/urdf/xacro/common_properties.xacro"/>
+  <xacro:include filename="$(find pomona_description)/urdf/pomona_original/xacro/common_properties.xacro"/>
   <!-- ── mobile base ──────────────────────────────────────────────────── -->
-  <xacro:include filename="$(find pomona_description)/urdf/xacro/scout_v2.xacro"/>
+  <xacro:include filename="$(find pomona_description)/urdf/pomona_original/xacro/scout_v2.xacro"/>
   <!-- ── mounting box (white cuboid carrying arm + display) ───────────── -->
-  <xacro:include filename="$(find pomona_description)/urdf/xacro/mount.xacro"/>
+  <xacro:include filename="$(find pomona_description)/urdf/pomona_original/xacro/mount.xacro"/>
   <!-- ── manipulator ──────────────────────────────────────────────────── -->
-  <xacro:include filename="$(find pomona_description)/urdf/xacro/xarm6.xacro"/>
+  <xacro:include filename="$(find pomona_description)/urdf/pomona_original/xacro/xarm6.xacro"/>
   <xacro:xarm6 prefix=""/>
   <!-- Mount xArm6 on Scout base: 0.212 forward of base centre, 0.26 up
@@ -35,5 +35,5 @@
   </joint>
   <!-- ── gripper ──────────────────────────────────────────────────────── -->
-  <xacro:include filename="$(find pomona_description)/urdf/xacro/ag95_gripper.xacro"/>
+  <xacro:include filename="$(find pomona_description)/urdf/pomona_original/xacro/ag95_gripper.xacro"/>
   <xacro:ag95_gripper prefix=""/>
   <!-- Attach AG95 base to xArm6 end-effector -->
@@ -44,11 +44,9 @@
   </joint>
   <!-- ── sensors (LiDAR, IMU, camera links) ───────────────────────────── -->
-  <xacro:include filename="$(find pomona_description)/urdf/xacro/sensors.xacro"/>
-  <!-- ── UVC lamp bar (front of box, below LiDAR) ─────────────────────── -->
-  <xacro:include filename="$(find pomona_description)/urdf/xacro/uvc_lamps.xacro"/>
+  <xacro:include filename="$(find pomona_description)/urdf/pomona_original/xacro/sensors.xacro"/>
   <!-- ── Gazebo plugins + ros2_control (conditional) ──────────────────── -->
   <xacro:if value="${use_sim}">
-    <xacro:include filename="$(find pomona_description)/urdf/xacro/gazebo_plugins.xacro"/>
-    <xacro:include filename="$(find pomona_description)/urdf/xacro/ros2_control.xacro"/>
+    <xacro:include filename="$(find pomona_description)/urdf/pomona_original/xacro/gazebo_plugins.xacro"/>
+    <xacro:include filename="$(find pomona_description)/urdf/pomona_original/xacro/ros2_control.xacro"/>
   </xacro:if>
 </robot>

File: src/pomona_description/urdf/pomona_original/xacro/scout_v2.xacro (robot description, xacro)
@@ -10,15 +10,21 @@
 -->
 <robot name="scout_v2" xmlns:xacro="http://ros.org/wiki/xacro">
-  <xacro:include filename="$(find pomona_description)/urdf/xacro/scout_wheel_type1.xacro"/>
-  <xacro:include filename="$(find pomona_description)/urdf/xacro/scout_wheel_type2.xacro"/>
+  <xacro:include filename="$(find pomona_description)/urdf/pomona_original/xacro/scout_wheel_type1.xacro"/>
+  <xacro:include filename="$(find pomona_description)/urdf/pomona_original/xacro/scout_wheel_type2.xacro"/>
   <!-- Vehicle Geometries -->
   <xacro:property name="base_x_size" value="0.9250"/>
   <xacro:property name="base_y_size" value="0.3800"/>
   <xacro:property name="base_z_size" value="0.2100"/>
+  <!-- Stock AgileX Scout V2 geometry (real-robot-accurate; BSD upstream). -->
   <xacro:property name="wheelbase" value="0.498"/>
   <xacro:property name="track"     value="0.58306"/>
   <xacro:property name="wheel_vertical_offset" value="-0.0702"/>
-  <xacro:property name="wheel_length" value="1.1653e-01"/>
-  <xacro:property name="wheel_radius" value="1.6459e-01"/>
+  <xacro:property name="wheel_length_stock" value="1.1653e-01"/>
+  <xacro:property name="wheel_radius_stock" value="1.6459e-01"/>
+  <!-- ORIGINAL model: wheels at stock size. The sim oversize knob (wheel_scale)
+       lives in the pomona_uvc model, not here. -->
+  <xacro:property name="wheel_scale"  value="1.0"/>
+  <xacro:property name="wheel_length" value="${wheel_length_stock * wheel_scale}"/>
+  <xacro:property name="wheel_radius" value="${wheel_radius_stock * wheel_scale}"/>
   <!-- Base link -->
   <link name="base_link">

File: src/pomona_description/urdf/pomona_original/xacro/scout_wheel_type1.xacro (robot description, xacro)
@@ -20,5 +20,5 @@
         <origin xyz="0 0 0" rpy="0 0 0"/>
         <geometry>
-          <mesh filename="package://pomona_description/meshes/wheels/wheel_type1.dae"/>
+          <mesh filename="package://pomona_description/meshes/wheels/wheel_type1.dae" scale="${wheel_scale} ${wheel_scale} ${wheel_scale}"/>
         </geometry>
       </visual>

File: src/pomona_description/urdf/pomona_uvc/xacro/scout_wheel_type1.xacro (robot description, xacro)
@@ -3,10 +3,10 @@
   Copyright 2026 Pravin Oli  <pravin.oli.08@gmail.com, olipravin18@gmail.com>
   Licensed under the Apache License, Version 2.0.
-  Adapted from agilexrobotics/scout_ros — scout_description/urdf/scout_wheel_type2.xacro
+  Adapted from agilexrobotics/scout_ros — scout_description/urdf/scout_wheel_type1.xacro
   Original: Copyright (c) 2015 Clearpath Robotics  /  Copyright (c) 2020 Weston Robot
   License : BSD-3-Clause
 -->
 <robot xmlns:xacro="http://ros.org/wiki/xacro" name="scout_wheel">
-  <xacro:macro name="scout_wheel_type2" params="wheel_prefix *joint_pose">
+  <xacro:macro name="scout_wheel_type1" params="wheel_prefix *joint_pose">
     <link name="${wheel_prefix}_wheel_link">
       <inertial>
@@ -20,5 +20,5 @@
         <origin xyz="0 0 0" rpy="0 0 0"/>
         <geometry>
-          <mesh filename="package://pomona_description/meshes/wheels/wheel_type2.dae"/>
+          <mesh filename="package://pomona_description/meshes/wheels/wheel_type1.dae" scale="${wheel_scale} ${wheel_scale} ${wheel_scale}"/>
         </geometry>
       </visual>
@@ -36,4 +36,5 @@
       <axis xyz="0 -1 0" rpy="0 0 0"/>
     </joint>
+    <!-- Friction for skid-steer -->
     <gazebo reference="${wheel_prefix}_wheel_link">
       <mu1>1.0</mu1>
