Commit message: fix(description): correct sim drivetrain wheel axis + per-pair wheel separation

File: src/pomona_description/urdf/pomona_original/urdf/pomona_original.urdf (robot description, URDF)
Before this commit: robot pomona, 31 links, 30 joints
Joints:
- joint front_left_wheel: axis 0 -1 0 -> 0 1 0
- joint rear_left_wheel: axis 0 -1 0 -> 0 1 0

File: src/pomona_description/urdf/pomona_original/urdf/pomona_original_sim.urdf (robot description, URDF)
Before this commit: robot pomona, 31 links, 30 joints
Joints:
- joint front_left_wheel: axis 0 -1 0 -> 0 1 0
- joint rear_left_wheel: axis 0 -1 0 -> 0 1 0

File: src/pomona_description/urdf/pomona_original/xacro/gazebo_plugins.xacro (robot description, xacro)
@@ -30,5 +30,12 @@
       <right_joint>front_right_wheel</right_joint>
       <right_joint>rear_right_wheel</right_joint>
+      <!-- ONE value per wheel pair (num_wheel_pairs=2). If only listed once,
+           pair 2 (rear wheels) silently falls back to the plugin default
+           (0.34 m / 0.2 m), so the rear axle turns with a different differential
+           than the front and the same-side wheels fight each other. Both pairs
+           share the Scout's track + wheel size, so repeat the same values. -->
       <wheel_separation>0.58306</wheel_separation>
+      <wheel_separation>0.58306</wheel_separation>
+      <wheel_diameter>${2 * wheel_radius}</wheel_diameter>
       <wheel_diameter>${2 * wheel_radius}</wheel_diameter>
       <max_wheel_torque>50.0</max_wheel_torque>

File: src/pomona_description/urdf/pomona_original/xacro/scout_v2.xacro (robot description, xacro)
@@ -70,5 +70,5 @@
   <!-- 4 wheels, counter-clockwise from front-right.
        Motors 1 & 2 (left side) are mechanically reversed. -->
-  <xacro:scout_wheel_type1 wheel_prefix="front_right">
+  <xacro:scout_wheel_type1 wheel_prefix="front_right" wheel_axis="0 -1 0">
     <origin xyz="${ wheelbase/2} ${-track/2} ${wheel_vertical_offset}" rpy="3.14 0 0"/>
   </xacro:scout_wheel_type1>
@@ -79,5 +79,5 @@
     <origin xyz="${-wheelbase/2} ${ track/2} ${wheel_vertical_offset}" rpy="0 0 0"/>
   </xacro:scout_wheel_type1>
-  <xacro:scout_wheel_type2 wheel_prefix="rear_right">
+  <xacro:scout_wheel_type2 wheel_prefix="rear_right" wheel_axis="0 -1 0">
     <origin xyz="${-wheelbase/2} ${-track/2} ${wheel_vertical_offset}" rpy="3.14 0 0"/>
   </xacro:scout_wheel_type2>

File: src/pomona_description/urdf/pomona_original/xacro/scout_wheel_type1.xacro (robot description, xacro)
@@ -8,5 +8,10 @@
 -->
 <robot xmlns:xacro="http://ros.org/wiki/xacro" name="scout_wheel">
-  <xacro:macro name="scout_wheel_type1" params="wheel_prefix *joint_pose">
+  <!-- wheel_axis: spin axis in the JOINT frame. Default ("0 1 0") suits the
+       unrolled left wheels. The right wheels carry a 180° roll (rpy="3.14 0 0")
+       that negates Y, so they must pass the NEGATED axis ("0 -1 0") to end up
+       with the SAME effective axis. If left/right effective axes differ the
+       diff-drive swaps linear<->angular; flipping all of them inverts fwd/back. -->
+  <xacro:macro name="scout_wheel_type1" params="wheel_prefix wheel_axis:='0 1 0' *joint_pose">
     <link name="${wheel_prefix}_wheel_link">
       <inertial>
@@ -34,5 +39,5 @@
       <child  link="${wheel_prefix}_wheel_link"/>
       <xacro:insert_block name="joint_pose"/>
-      <axis xyz="0 -1 0" rpy="0 0 0"/>
+      <axis xyz="${wheel_axis}" rpy="0 0 0"/>
     </joint>
     <!-- Friction for skid-steer -->

File: src/pomona_description/urdf/pomona_original/xacro/scout_wheel_type2.xacro (robot description, xacro)
@@ -8,5 +8,10 @@
 -->
 <robot xmlns:xacro="http://ros.org/wiki/xacro" name="scout_wheel">
-  <xacro:macro name="scout_wheel_type2" params="wheel_prefix *joint_pose">
+  <!-- wheel_axis: spin axis in the JOINT frame. Default ("0 1 0") suits the
+       unrolled left wheels. The right wheels carry a 180° roll (rpy="3.14 0 0")
+       that negates Y, so they must pass the NEGATED axis ("0 -1 0") to end up
+       with the SAME effective axis. If left/right effective axes differ the
+       diff-drive swaps linear<->angular; flipping all of them inverts fwd/back. -->
+  <xacro:macro name="scout_wheel_type2" params="wheel_prefix wheel_axis:='0 1 0' *joint_pose">
     <link name="${wheel_prefix}_wheel_link">
       <inertial>
@@ -34,5 +39,5 @@
       <child  link="${wheel_prefix}_wheel_link"/>
       <xacro:insert_block name="joint_pose"/>
-      <axis xyz="0 -1 0" rpy="0 0 0"/>
+      <axis xyz="${wheel_axis}" rpy="0 0 0"/>
     </joint>
     <gazebo reference="${wheel_prefix}_wheel_link">

File: src/pomona_description/urdf/pomona_uvc/urdf/pomona_uvc.urdf (robot description, URDF)
Before this commit: robot pomona, 14 links, 13 joints
Joints:
- joint front_left_wheel: axis 0 -1 0 -> 0 1 0
- joint rear_left_wheel: axis 0 -1 0 -> 0 1 0

File: src/pomona_description/urdf/pomona_uvc/urdf/pomona_uvc_sim.urdf (robot description, URDF)
Before this commit: robot pomona, 14 links, 13 joints
Joints:
- joint front_left_wheel: axis 0 -1 0 -> 0 1 0
- joint rear_left_wheel: axis 0 -1 0 -> 0 1 0

File: src/pomona_description/urdf/pomona_uvc/xacro/gazebo_plugins.xacro (robot description, xacro)
@@ -28,5 +28,12 @@
       <right_joint>front_right_wheel</right_joint>
       <right_joint>rear_right_wheel</right_joint>
+      <!-- ONE value per wheel pair (num_wheel_pairs=2). If only listed once,
+           pair 2 (rear wheels) silently falls back to the plugin default
+           (0.34 m / 0.2 m), so the rear axle turns with a different differential
+           than the front and the same-side wheels fight each other. Both pairs
+           share the Scout's track + wheel size, so repeat the same values. -->
       <wheel_separation>0.58306</wheel_separation>
+      <wheel_separation>0.58306</wheel_separation>
+      <wheel_diameter>${2 * wheel_radius}</wheel_diameter>
       <wheel_diameter>${2 * wheel_radius}</wheel_diameter>
       <max_wheel_torque>50.0</max_wheel_torque>

File: src/pomona_description/urdf/pomona_uvc/xacro/scout_v2.xacro (robot description, xacro)
@@ -70,5 +70,5 @@
   <!-- 4 wheels, counter-clockwise from front-right.
        Motors 1 & 2 (left side) are mechanically reversed. -->
-  <xacro:scout_wheel_type1 wheel_prefix="front_right">
+  <xacro:scout_wheel_type1 wheel_prefix="front_right" wheel_axis="0 -1 0">
     <origin xyz="${ wheelbase/2} ${-track/2} ${wheel_vertical_offset}" rpy="3.14 0 0"/>
   </xacro:scout_wheel_type1>
@@ -79,5 +79,5 @@
     <origin xyz="${-wheelbase/2} ${ track/2} ${wheel_vertical_offset}" rpy="0 0 0"/>
   </xacro:scout_wheel_type1>
-  <xacro:scout_wheel_type2 wheel_prefix="rear_right">
+  <xacro:scout_wheel_type2 wheel_prefix="rear_right" wheel_axis="0 -1 0">
     <origin xyz="${-wheelbase/2} ${-track/2} ${wheel_vertical_offset}" rpy="3.14 0 0"/>
   </xacro:scout_wheel_type2>

Commit message: fix(description): TF root, wheel joint states, lidar self-returns; UV-C beam viz

File: src/pomona_description/urdf/pomona_original/urdf/pomona_original.urdf (robot description, URDF)
Before this commit: robot pomona, 31 links, 30 joints
Joints:
- joint base_footprint_joint: child base_footprint -> base_link; origin xyz=0 0 -0.23479 rpy=0 0 0 -> xyz=0 0 0.23479 rpy=0 0 0; parent base_link -> base_footprint

File: src/pomona_description/urdf/pomona_original/urdf/pomona_original_sim.urdf (robot description, URDF)
Before this commit: robot pomona, 31 links, 30 joints
Joints:
- joint base_footprint_joint: child base_footprint -> base_link; origin xyz=0 0 -0.23479 rpy=0 0 0 -> xyz=0 0 0.23479 rpy=0 0 0; parent base_link -> base_footprint

File: src/pomona_description/urdf/pomona_original/xacro/gazebo_plugins.xacro (robot description, xacro)
@@ -7,5 +7,6 @@
   Plugins:
     - libgazebo_ros_diff_drive.so       — Scout V2 skid-steer (4 wheels)
-    - libgazebo_ros_joint_state_publisher.so — joint_states for arm + gripper
+    - libgazebo_ros_joint_state_publisher.so — joint_states for the 4 wheels
+                                               (arm+gripper come from ros2_control)
     - libgazebo_ros_ray_sensor.so       — rslidar (gpu_ray) → /scan
     - libgazebo_ros_camera.so           — D435 RGB + depth
@@ -50,7 +51,20 @@
       <update_rate>50.0</update_rate>
     </plugin>
-    <!-- NOTE: arm/gripper joint_states are published by joint_state_broadcaster
-         (ros2_control.xacro), not by libgazebo_ros_joint_state_publisher, to
-         avoid two publishers racing on /joint_states. -->
+    <!-- arm/gripper joint_states come from joint_state_broadcaster
+         (ros2_control.xacro). The wheels are NOT in ros2_control and the
+         diff_drive plugin doesn't publish their positions, so they need their
+         own publisher or robot_state_publisher can't place them (wheels float
+         at the origin in RViz). Listing ONLY the 4 wheels keeps this disjoint
+         from the broadcaster (arm+gripper) — no two publishers on one joint. -->
+    <plugin name="wheel_joint_state" filename="libgazebo_ros_joint_state_publisher.so">
+      <ros>
+        <remapping>~/out:=joint_states</remapping>
+      </ros>
+      <update_rate>30</update_rate>
+      <joint_name>front_left_wheel</joint_name>
+      <joint_name>front_right_wheel</joint_name>
+      <joint_name>rear_left_wheel</joint_name>
+      <joint_name>rear_right_wheel</joint_name>
+    </plugin>
   </gazebo>
   <!-- ════════════════════════════════════════════════════════════════════
@@ -69,8 +83,15 @@
         <scan>
           <horizontal>
-            <samples>720</samples>
+            <!-- 240 deg forward arc (NOT full 360): the lidar sits embedded low
+                 inside box_link (front wall 0.07 m ahead, sides 0.16 m -> both
+                 within the 0.2 m min_range, so ignored), but the REAR of the box
+                 + display panel are >0.2 m back and would otherwise be mapped as
+                 a rectangle trailing the robot. Trimming the rear ~120 deg drops
+                 those self-returns while keeping the low plane. (Proper 360 deg
+                 needs a mast-mounted/3D lidar.) -->
+            <samples>600</samples>
             <resolution>1</resolution>
-            <min_angle>-3.14159</min_angle>
-            <max_angle>3.14159</max_angle>
+            <min_angle>-2.10</min_angle>
+            <max_angle>2.10</max_angle>
           </horizontal>
         </scan>

File: src/pomona_description/urdf/pomona_original/xacro/scout_v2.xacro (robot description, xacro)
@@ -48,9 +48,14 @@
     </collision>
   </link>
+  <!-- base_footprint is the TF root (on the ground): the Gazebo diff_drive
+       plugin publishes odom -> base_footprint, so base_footprint must be the
+       parent of base_link. If this joint is inverted (base_link -> footprint),
+       base_footprint ends up with two parents (odom + base_link) and the TF
+       tree breaks -> slam_toolbox drops every scan ("queue is full"). -->
   <link name="base_footprint"/>
   <joint name="base_footprint_joint" type="fixed">
-    <origin xyz="0 0 ${wheel_vertical_offset - wheel_radius}" rpy="0 0 0"/>
-    <parent link="base_link"/>
-    <child  link="base_footprint"/>
+    <origin xyz="0 0 ${wheel_radius - wheel_vertical_offset}" rpy="0 0 0"/>
+    <parent link="base_footprint"/>
+    <child  link="base_link"/>
   </joint>
   <link name="inertial_link">

File: src/pomona_description/urdf/pomona_uvc/urdf/pomona_uvc.urdf (robot description, URDF)
Before this commit: robot pomona, 18 links, 17 joints
Links:
- added link uvc_beam_link, mass 0.001; visual box size=0.6935 0.9 0.616; visual box size=0.6935 0.9 0.616
Joints:
- added joint uvc_beam_joint: type fixed, parent base_link, child uvc_beam_link, origin xyz=0 0 0 rpy=0 0 0
- joint base_footprint_joint: child base_footprint -> base_link; origin xyz=0 0 -0.23479 rpy=0 0 0 -> xyz=0 0 0.23479 rpy=0 0 0; parent base_link -> base_footprint

File: src/pomona_description/urdf/pomona_uvc/urdf/pomona_uvc_sim.urdf (robot description, URDF)
Before this commit: robot pomona, 18 links, 17 joints
Links:
- added link uvc_beam_link, mass 0.001; visual box size=0.6935 0.9 0.616; visual box size=0.6935 0.9 0.616
Joints:
- added joint uvc_beam_joint: type fixed, parent base_link, child uvc_beam_link, origin xyz=0 0 0 rpy=0 0 0
- joint base_footprint_joint: child base_footprint -> base_link; origin xyz=0 0 -0.23479 rpy=0 0 0 -> xyz=0 0 0.23479 rpy=0 0 0; parent base_link -> base_footprint

File: src/pomona_description/urdf/pomona_uvc/xacro/common_properties.xacro (robot description, xacro)
@@ -21,4 +21,8 @@
   <material name="orange"><color rgba="1.0 0.424 0.039 1.0"/></material>
   <material name="brown"><color rgba="0.871 0.812 0.765 1.0"/></material>
+  <!-- UV-C lamp "on" violet + translucent projected beam (RViz; Gazebo overrides
+       these with Gazebo/PurpleGlow + Gazebo/DarkMagentaTransparent). -->
+  <material name="uvc_violet"><color rgba="0.60 0.10 0.95 1.0"/></material>
+  <material name="uvc_beam"><color rgba="0.60 0.15 0.95 0.22"/></material>
   <!-- Constants -->
   <xacro:property name="M_PI" value="3.14159"/>

File: src/pomona_description/urdf/pomona_uvc/xacro/gazebo_plugins.xacro (robot description, xacro)
@@ -48,10 +48,27 @@
       <update_rate>50.0</update_rate>
     </plugin>
-    <!-- NOTE: arm/gripper joint_states are published by joint_state_broadcaster
-         (ros2_control.xacro), not by libgazebo_ros_joint_state_publisher, to
-         avoid two publishers racing on /joint_states. -->
+    <!-- Wheel joint states. The diff_drive plugin spins the wheels in Gazebo
+         but does NOT publish their joint positions, and the wheels are not part
+         of ros2_control. Without this, robot_state_publisher has no angle for
+         the 4 continuous wheel joints and the wheels float at the origin in
+         RViz. pomona_original needs the same plugin (wheels only — disjoint
+         from joint_state_broadcaster, which covers arm+gripper, so no race). -->
+    <plugin name="wheel_joint_state" filename="libgazebo_ros_joint_state_publisher.so">
+      <ros>
+        <remapping>~/out:=joint_states</remapping>
+      </ros>
+      <update_rate>30</update_rate>
+      <joint_name>front_left_wheel</joint_name>
+      <joint_name>front_right_wheel</joint_name>
+      <joint_name>rear_left_wheel</joint_name>
+      <joint_name>rear_right_wheel</joint_name>
+    </plugin>
   </gazebo>
   <!-- ════════════════════════════════════════════════════════════════════
-       Robosense LiDAR (publishes /scan via ray_sensor)
+       Robosense LiDAR — 360° 2D plane (publishes /scan_raw via ray_sensor)
+       A laser_self_filter node (pomona_state_publisher_uvc.launch.py) drops the
+       self-returns (the low plane clips the rear display) and republishes /scan,
+       so the robot body reads as free space, not a phantom obstacle. Full 360°
+       is kept — no angular trim — because the filter is geometric, not by angle.
        ════════════════════════════════════════════════════════════════════ -->
   <gazebo reference="rslidar">
@@ -74,5 +91,9 @@
         </scan>
         <range>
-          <min>0.2</min>
+          <!-- 0.1 m: halves the old 0.2 m near-field dead disc (the front-middle
+               gap that stayed unexplored as the robot advanced) without pulling
+               in so far that the gpu_ray catches the sensor housing / box top
+               (0.05 m did). -->
+          <min>0.1</min>
           <max>5.0</max>
           <resolution>0.01</resolution>
@@ -81,5 +102,5 @@
       <plugin name="rslidar_controller" filename="libgazebo_ros_ray_sensor.so">
         <ros>
-          <remapping>~/out:=scan</remapping>
+          <remapping>~/out:=scan_raw</remapping>
         </ros>
         <output_type>sensor_msgs/LaserScan</output_type>
@@ -105,9 +126,19 @@
   </gazebo>
   <!-- ════════════════════════════════════════════════════════════════════
-       UV-C lamp tubes — colour the whole lamp link blue in Gazebo
-       (URDF <material name="blue"> is ignored by Gazebo; needs a Gazebo/ script)
+       UV-C lamp tubes — emissive violet so the lamps read as ON.
+       (URDF <material> is ignored by Gazebo; needs a Gazebo/ script. PurpleGlow
+       is an emissive built-in → the tubes glow like energised UV-C lamps.)
        ════════════════════════════════════════════════════════════════════ -->
   <gazebo reference="uvc_lamps_link">
-    <material>Gazebo/Blue</material>
+    <material>Gazebo/PurpleGlow</material>
+  </gazebo>
+  <!-- ════════════════════════════════════════════════════════════════════
+       UV-C projected beam — translucent violet "light curtain" volume from the
+       lamps down onto the bed. A continuous rendered volume (not discrete rays
+       like the lidar). DarkMagentaTransparent is alpha-blended so the beds show
+       through, tinted violet where the UV-C lands.
+       ════════════════════════════════════════════════════════════════════ -->
+  <gazebo reference="uvc_beam_link">
+    <material>Gazebo/DarkMagentaTransparent</material>
   </gazebo>
   <!-- ════════════════════════════════════════════════════════════════════

File: src/pomona_description/urdf/pomona_uvc/xacro/scout_v2.xacro (robot description, xacro)
@@ -48,9 +48,14 @@
     </collision>
   </link>
+  <!-- base_footprint is the TF root (on the ground): the Gazebo diff_drive
+       plugin publishes odom -> base_footprint, so base_footprint must be the
+       parent of base_link. If this joint is inverted (base_link -> footprint),
+       base_footprint ends up with two parents (odom + base_link) and the TF
+       tree breaks -> slam_toolbox drops every scan ("queue is full"). -->
   <link name="base_footprint"/>
   <joint name="base_footprint_joint" type="fixed">
-    <origin xyz="0 0 ${wheel_vertical_offset - wheel_radius}" rpy="0 0 0"/>
-    <parent link="base_link"/>
-    <child  link="base_footprint"/>
+    <origin xyz="0 0 ${wheel_radius - wheel_vertical_offset}" rpy="0 0 0"/>
+    <parent link="base_footprint"/>
+    <child  link="base_link"/>
   </joint>
   <link name="inertial_link">

File: src/pomona_description/urdf/pomona_uvc/xacro/sensors.xacro (robot description, xacro)
@@ -16,4 +16,8 @@
        above the base centre. Mounted on box_link with the original
        laser_Link transform from scout_xarm_base (xyz 0.37655 0 0.003).
+       Low (~0.351 m AGL) on purpose: the single 2D plane then clips the
+       0.40 m bed side-walls so the furrows map as corridors. (We tried a
+       raised central 3D lidar, but its downward rings scanned the robot's
+       own rear display as a phantom obstacle — reverted to this 2D mount.)
        Visual uses the ported laser_link mesh; collision is a cheap cylinder.
        ════════════════════════════════════════════════════════════════════ -->

File: src/pomona_description/urdf/pomona_uvc/xacro/uvc_cantilever.xacro (robot description, xacro)
@@ -60,5 +60,5 @@
   <xacro:property name="panel_x_c"   value="0.065"/>   <!-- panel fore-aft centre (= box centre) -->
   <xacro:property name="panel_thick" value="0.012"/>   <!-- panel thickness (Z) — thin flat plate -->
-  <xacro:property name="rod_x"       value="0.212"/>   <!-- mast over the arm base -->
+  <xacro:property name="rod_x"       value="0.065"/>   <!-- mast at box/panel fore-aft centre (= panel_x_c); cross-tube now welds each panel at the MIDPOINT of its inner edge. (Was 0.212 over the arm base, which welded 0.147 m forward of centre; the arm-base mesh at 0.212 is now the lidar pedestal.) -->
   <xacro:property name="rod_z_bot"   value="0.28"/>
   <xacro:property name="rod_radius"  value="0.025"/>   <!-- circular mast + cross-tube radius -->
@@ -82,4 +82,11 @@
   <xacro:property name="flap_thick"   value="0.006"/>  <!-- thin shield plate -->
   <xacro:property name="lamp_z" value="${arm_z - panel_thick/2 - tube_radius - 0.004}"/>
+  <!-- UV-C projected beam: a translucent "light curtain" volume from the lamp
+       plane down onto the bed top, so the disinfection looks ON in Gazebo (a
+       continuous rendered violet volume, not discrete rays). Bed top is 0.40 m
+       AGL; base_link sits 0.235 m AGL → bed top = 0.165 in base_link. -->
+  <xacro:property name="bed_top_z" value="0.165"/>
+  <xacro:property name="beam_h"  value="${lamp_z - bed_top_z}"/>
+  <xacro:property name="beam_cz" value="${(lamp_z + bed_top_z)/2.0}"/>
   <!-- housing for one side: flat roof plate + two thin side flaps (skirts) that
        hang down on both long edges so the UV-C only projects onto the bed -->
@@ -114,5 +121,5 @@
                 rpy="1.5708 0 0"/>
         <geometry><cylinder radius="${tube_radius}" length="${tube_len}"/></geometry>
-        <material name="blue"/>
+        <material name="uvc_violet"/>
       </visual>
       <xacro:uvc_tube_row name="${name}" side="${side}" i="${i+1}" n="${n}"/>
@@ -206,4 +213,29 @@
     <parent link="base_link"/>
     <child  link="uvc_lamps_link"/>
+    <origin xyz="0 0 0" rpy="0 0 0"/>
+  </joint>
+  <!-- ── UV-C beam link: translucent projected "light curtain" under each panel
+       (Gazebo colours it Gazebo/DarkMagentaTransparent). Visual only — no
+       collision (it is light, not a solid). ── -->
+  <link name="uvc_beam_link">
+    <visual name="uvc_beam_left">
+      <origin xyz="${panel_x_c} ${panel_y_c} ${beam_cz}" rpy="0 0 0"/>
+      <geometry><box size="${panel_len*0.95} ${tube_len} ${beam_h}"/></geometry>
+      <material name="uvc_beam"/>
+    </visual>
+    <visual name="uvc_beam_right">
+      <origin xyz="${panel_x_c} ${-panel_y_c} ${beam_cz}" rpy="0 0 0"/>
+      <geometry><box size="${panel_len*0.95} ${tube_len} ${beam_h}"/></geometry>
+      <material name="uvc_beam"/>
+    </visual>
+    <inertial>
+      <origin xyz="${panel_x_c} 0 ${beam_cz}" rpy="0 0 0"/>
+      <mass value="0.001"/>
+      <inertia ixx="1e-6" ixy="0" ixz="0" iyy="1e-6" iyz="0" izz="1e-6"/>
+    </inertial>
+  </link>
+  <joint name="uvc_beam_joint" type="fixed">
+    <parent link="base_link"/>
+    <child  link="uvc_beam_link"/>
     <origin xyz="0 0 0" rpy="0 0 0"/>
   </joint>
