Commit message: feat(uvc): redesign UV-C boom — T-frame, row-wise blue lamps, shield flaps, 2 D455 cameras

File: src/pomona_description/urdf/pomona_uvc/urdf/pomona_uvc.urdf (robot description, URDF)
Before this commit: robot pomona, 14 links, 13 joints
Links:
- added link uvc_cam_left_link; collision box size=0.124 0.029 0.026; visual mesh filename=package://pomona_description/meshes/sensors/d455.stl scale=0.001 0.001 0.001
- added link uvc_cam_left_optical_frame
- added link uvc_cam_right_link; collision box size=0.124 0.029 0.026; visual mesh filename=package://pomona_description/meshes/sensors/d455.stl scale=0.001 0.001 0.001
- added link uvc_cam_right_optical_frame
- link uvc_cantilever_link: geometry collision box size=0.09 0.07 0.062; collision box size=0.09 0.07 0.062
- link uvc_lamps_link: geometry collision box size=0.73 0.9 0.018; collision box size=0.73 0.9 0.018
Joints:
- added joint uvc_cam_left_joint: type fixed, parent base_link, child uvc_cam_left_link, origin xyz=0.53 1.0 0.74 rpy=0 1.5708 0
- added joint uvc_cam_left_optical_joint: type fixed, parent uvc_cam_left_link, child uvc_cam_left_optical_frame, origin xyz=0 0 0 rpy=-1.5708 0 -1.5708
- added joint uvc_cam_right_joint: type fixed, parent base_link, child uvc_cam_right_link, origin xyz=0.53 -1.0 0.74 rpy=0 1.5708 0
- added joint uvc_cam_right_optical_joint: type fixed, parent uvc_cam_right_link, child uvc_cam_right_optical_frame, origin xyz=0 0 0 rpy=-1.5708 0 -1.5708

File: src/pomona_description/urdf/pomona_uvc/urdf/pomona_uvc_sim.urdf (robot description, URDF)
Before this commit: robot pomona, 14 links, 13 joints
Links:
- added link uvc_cam_left_link; collision box size=0.124 0.029 0.026; visual mesh filename=package://pomona_description/meshes/sensors/d455.stl scale=0.001 0.001 0.001
- added link uvc_cam_left_optical_frame
- added link uvc_cam_right_link; collision box size=0.124 0.029 0.026; visual mesh filename=package://pomona_description/meshes/sensors/d455.stl scale=0.001 0.001 0.001
- added link uvc_cam_right_optical_frame
- link uvc_cantilever_link: geometry collision box size=0.09 0.07 0.062; collision box size=0.09 0.07 0.062
- link uvc_lamps_link: geometry collision box size=0.73 0.9 0.018; collision box size=0.73 0.9 0.018
Joints:
- added joint uvc_cam_left_joint: type fixed, parent base_link, child uvc_cam_left_link, origin xyz=0.53 1.0 0.74 rpy=0 1.5708 0
- added joint uvc_cam_left_optical_joint: type fixed, parent uvc_cam_left_link, child uvc_cam_left_optical_frame, origin xyz=0 0 0 rpy=-1.5708 0 -1.5708
- added joint uvc_cam_right_joint: type fixed, parent base_link, child uvc_cam_right_link, origin xyz=0.53 -1.0 0.74 rpy=0 1.5708 0
- added joint uvc_cam_right_optical_joint: type fixed, parent uvc_cam_right_link, child uvc_cam_right_optical_frame, origin xyz=0 0 0 rpy=-1.5708 0 -1.5708

File: src/pomona_description/urdf/pomona_uvc/xacro/gazebo_plugins.xacro (robot description, xacro)
@@ -75,5 +75,5 @@
         <range>
           <min>0.2</min>
-          <max>30.0</max>
+          <max>5.0</max>
           <resolution>0.01</resolution>
         </range>
@@ -104,3 +104,59 @@
     </sensor>
   </gazebo>
+  <!-- ════════════════════════════════════════════════════════════════════
+       UV-C lamp tubes — colour the whole lamp link blue in Gazebo
+       (URDF <material name="blue"> is ignored by Gazebo; needs a Gazebo/ script)
+       ════════════════════════════════════════════════════════════════════ -->
+  <gazebo reference="uvc_lamps_link">
+    <material>Gazebo/Blue</material>
+  </gazebo>
+  <!-- ════════════════════════════════════════════════════════════════════
+       RealSense D455 x2 — one per panel, looking down at each bed
+       -> /uvc_cam_left/{color,depth}/*  and  /uvc_cam_right/{color,depth}/*
+       ════════════════════════════════════════════════════════════════════ -->
+  <xacro:macro name="uvc_cam_gazebo" params="name">
+    <gazebo reference="uvc_cam_${name}_link">
+      <sensor name="uvc_cam_${name}_rgb" type="camera">
+        <always_on>true</always_on>
+        <visualize>false</visualize>
+        <update_rate>15</update_rate>
+        <camera>
+          <horizontal_fov>1.5708</horizontal_fov>
+          <image><width>640</width><height>480</height><format>R8G8B8</format></image>
+          <clip><near>0.1</near><far>6.0</far></clip>
+        </camera>
+        <plugin name="uvc_cam_${name}_rgb_ctrl" filename="libgazebo_ros_camera.so">
+          <ros>
+            <namespace>/uvc_cam_${name}</namespace>
+            <remapping>image_raw:=color/image_raw</remapping>
+            <remapping>camera_info:=color/camera_info</remapping>
+          </ros>
+          <frame_name>uvc_cam_${name}_optical_frame</frame_name>
+        </plugin>
+      </sensor>
+      <sensor name="uvc_cam_${name}_depth" type="depth">
+        <always_on>true</always_on>
+        <visualize>false</visualize>
+        <update_rate>10</update_rate>
+        <camera>
+          <horizontal_fov>1.518</horizontal_fov>
+          <image><width>424</width><height>240</height></image>
+          <clip><near>0.2</near><far>6.0</far></clip>
+        </camera>
+        <plugin name="uvc_cam_${name}_depth_ctrl" filename="libgazebo_ros_camera.so">
+          <ros>
+            <namespace>/uvc_cam_${name}</namespace>
+            <remapping>image_raw:=depth/image_rect_raw</remapping>
+            <remapping>camera_info:=depth/camera_info</remapping>
+            <remapping>points:=depth/points</remapping>
+          </ros>
+          <frame_name>uvc_cam_${name}_optical_frame</frame_name>
+          <point_cloud_cutoff>0.2</point_cloud_cutoff>
+          <point_cloud_cutoff_max>6.0</point_cloud_cutoff_max>
+        </plugin>
+      </sensor>
+    </gazebo>
+  </xacro:macro>
+  <xacro:uvc_cam_gazebo name="left"/>
+  <xacro:uvc_cam_gazebo name="right"/>
 </robot>

File: src/pomona_description/urdf/pomona_uvc/xacro/uvc_cantilever.xacro (robot description, xacro)
@@ -4,20 +4,30 @@
   Licensed under the Apache License, Version 2.0.
   UV-C cantilever (pomona_uvc only) — replaces the xArm6 arm.
-  Shape (top view):
-      [====panel_L====]            [====panel_R====]
-              \                            /
-               +============o============+
-                            ^ base/rod on the box
-  center 'o' = base/rod on the box; a cross-arm reaches out to each side; at
-  each end a FLAT, THIN horizontal panel spans a full strawberry bed and holds
-  4 fore-aft UV-C lamp tubes pointing down.
-  Bed coverage (per side, from robot centreline):
-    near edge ~0.40 m (= outer wheel edge) ... far edge ~1.10 m  -> 0.70 m bed,
-    panel centred at 0.75 m. Robot drives the furrow between two beds.
-  Two links: uvc_cantilever_link (rod + arm + panels, grey) and uvc_lamps_link
-  (tubes only, so Gazebo colours just the lamps blue — see gazebo_plugins.xacro).
-  Primitives only (no CAD). base_link frame; with stock wheels the ground is at
-  base_link z = -0.235, so arm_z = 0.50 -> panels ~0.735 m AGL, base mount
-  (z=0.26) is ~0.495 m AGL.
+  T-frame (front view):
+       panel_L                 mast                 panel_R
+      [=======]                 |                  [=======]
+       | | | |  <- lamps        |          lamps -> | | | |
+              \                 |                  /
+               +=== cross-tube ===o=== cross-tube ===+   (T-weld at mast top)
+                                  |
+                                (base/rod on the box)
+  A vertical CIRCULAR mast carries one horizontal CIRCULAR cross-tube (same dia),
+  T-welded at the top. The cross-tube reaches out to the INNER EDGE of each flat
+  panel (weld gusset there); each 1 m-wide panel cantilevers outward over a full
+  strawberry bed. Beds are 2 m centre-to-centre; the robot drives the 1 m furrow
+  between them.
+  Each panel = a shallow housing: flat roof plate + two side shield FLAPS hanging
+  down on both long edges (skirt_depth) so the UV-C only projects onto the bed.
+  Lamps = n_tubes thin blue glass cylinders running ACROSS the bed (row-wise),
+  spread along the driving direction, recessed under the roof.
+  A RealSense D455 (official mesh, meshes/sensors/d455.stl) hangs on a small
+  L-bracket FORWARD of and below each panel front edge, lens looking straight
+  down at its bed -> /uvc_cam_{left,right}/{color,depth}/* (gazebo_plugins.xacro).
+  Links: uvc_cantilever_link (mast + cross-tube + gussets + panels + flaps +
+  brackets, grey), uvc_lamps_link (tubes only -> coloured blue in Gazebo), and
+  uvc_cam_{left,right}_link (D455). Primitives + the D455 mesh; base_link frame.
+  Stock wheels -> ground at base_link z = -0.235, so arm_z = 0.80 -> panels
+  ~1.08 m AGL. All sizes are the tunables below; after editing, regenerate with
+  scripts/xacro_to_urdf.sh (+ gz sdf for models/pomona_uvc/model.sdf).
 -->
 <robot xmlns:xacro="http://ros.org/wiki/xacro">
@@ -44,20 +54,34 @@
   </joint>
   <!-- ── tunables (base_link frame) ────────────────────────────────────── -->
-  <xacro:property name="panel_y_c"   value="0.75"/>    <!-- panel centre (bed centre) from centreline -->
-  <xacro:property name="panel_width" value="0.70"/>    <!-- panel lateral width (Y) = bed width -->
-  <xacro:property name="arm_z"       value="0.50"/>    <!-- panel plane height (~0.78 m AGL) -->
+  <xacro:property name="panel_y_c"   value="1.0"/>    <!-- panel centre (bed centre) from centreline -->
+  <xacro:property name="panel_width" value="1.0"/>    <!-- panel lateral width (Y) = bed width -->
+  <xacro:property name="arm_z"       value="0.80"/>    <!-- panel plane height (~1.08 m AGL (+0.30 m)) -->
   <xacro:property name="panel_len"   value="0.73"/>    <!-- panel fore-aft length (= box length) -->
   <xacro:property name="panel_x_c"   value="0.065"/>   <!-- panel fore-aft centre (= box centre) -->
   <xacro:property name="panel_thick" value="0.012"/>   <!-- panel thickness (Z) — thin flat plate -->
-  <xacro:property name="beam_w"      value="0.035"/>   <!-- cross-arm square section -->
   <xacro:property name="rod_x"       value="0.212"/>   <!-- mast over the arm base -->
   <xacro:property name="rod_z_bot"   value="0.28"/>
-  <xacro:property name="rod_radius"  value="0.025"/>
-  <xacro:property name="tube_radius" value="0.008"/>   <!-- thin UV-C tube (~16 mm dia) -->
-  <!-- 4 tubes per side, spread across the bed width (offsets from panel centre) -->
-  <xacro:property name="tube_o1" value="0.27"/>
-  <xacro:property name="tube_o2" value="0.09"/>
-  <xacro:property name="lamp_z" value="${arm_z - panel_thick/2 - tube_radius}"/>
-  <!-- a flat, thin horizontal panel (grey) on one side -->
+  <xacro:property name="rod_radius"  value="0.025"/>   <!-- circular mast + cross-tube radius -->
+  <!-- T-frame: a single horizontal CIRCULAR cross-tube (same dia as the mast)
+       welded to the mast top, reaching out to the INNER EDGE of each panel.
+       Panels cantilever outward from that inner-edge weld (not the centre). -->
+  <xacro:property name="panel_inner" value="${panel_y_c - panel_width/2}"/>  <!-- inner long edge (0.5) -->
+  <xacro:property name="panel_front_x" value="${panel_x_c + panel_len/2}"/>  <!-- leading (front) edge in +X -->
+  <!-- D455 camera: on an L-bracket FORWARD of the panel front edge, hanging
+       below it, lens looking straight down at the bed (clear of the lamps) -->
+  <xacro:property name="cam_scale" value="0.001"/>   <!-- D455 STL is in mm -->
+  <xacro:property name="cam_fwd"   value="0.10"/>    <!-- forward of the panel front edge -->
+  <xacro:property name="cam_drop"  value="0.06"/>    <!-- 6 cm drop -->
+  <!-- UV-C lamps: thin cylindrical glass tubes running ACROSS the bed (row-wise),
+       several spread along the driving direction, recessed in a shallow housing -->
+  <xacro:property name="tube_radius"  value="0.009"/>  <!-- ~18 mm dia glass tube (realistic) -->
+  <xacro:property name="n_tubes"      value="6"/>      <!-- lamps per panel -->
+  <xacro:property name="tube_len"     value="${panel_width - 0.10}"/>  <!-- across bed, inside the flaps -->
+  <xacro:property name="tube_inset_x" value="0.08"/>   <!-- keep end lamps inside the panel ends -->
+  <xacro:property name="skirt_depth"  value="0.18"/>   <!-- side flap hang-down (shields stray rays) -->
+  <xacro:property name="flap_thick"   value="0.006"/>  <!-- thin shield plate -->
+  <xacro:property name="lamp_z" value="${arm_z - panel_thick/2 - tube_radius - 0.004}"/>
+  <!-- housing for one side: flat roof plate + two thin side flaps (skirts) that
+       hang down on both long edges so the UV-C only projects onto the bed -->
   <xacro:macro name="uvc_panel" params="name side">
     <visual name="${name}_panel">
@@ -70,22 +94,35 @@
       <geometry><box size="${panel_len} ${panel_width} ${panel_thick}"/></geometry>
     </collision>
-  </xacro:macro>
-  <!-- one fore-aft UV-C tube (blue) at an absolute Y -->
-  <xacro:macro name="uvc_tube" params="name y">
-    <visual name="uvc_lamp_${name}">
-      <origin xyz="${panel_x_c} ${y} ${lamp_z}" rpy="0 1.5708 0"/>
-      <geometry><cylinder radius="${tube_radius}" length="${panel_len}"/></geometry>
-      <material name="blue"/>
-    </visual>
-  </xacro:macro>
-  <!-- 4 tubes + one collision box, for one side -->
+    <!-- inner-edge shield flap -->
+    <visual name="${name}_flap_in">
+      <origin xyz="${panel_x_c} ${side*(panel_y_c - panel_width/2)} ${arm_z - skirt_depth/2}" rpy="0 0 0"/>
+      <geometry><box size="${panel_len} ${flap_thick} ${skirt_depth}"/></geometry>
+      <material name="grey"/>
+    </visual>
+    <!-- outer-edge shield flap -->
+    <visual name="${name}_flap_out">
+      <origin xyz="${panel_x_c} ${side*(panel_y_c + panel_width/2)} ${arm_z - skirt_depth/2}" rpy="0 0 0"/>
+      <geometry><box size="${panel_len} ${flap_thick} ${skirt_depth}"/></geometry>
+      <material name="grey"/>
+    </visual>
+  </xacro:macro>
+  <!-- recursive: place n cross-bed (row-wise) glass tubes spread along +X -->
+  <xacro:macro name="uvc_tube_row" params="name side i n">
+    <xacro:if value="${i &lt; n}">
+      <visual name="uvc_lamp_${name}_${i}">
+        <origin xyz="${panel_x_c - panel_len/2 + tube_inset_x + i*(panel_len - 2*tube_inset_x)/(n-1)} ${side*panel_y_c} ${lamp_z}"
+                rpy="1.5708 0 0"/>
+        <geometry><cylinder radius="${tube_radius}" length="${tube_len}"/></geometry>
+        <material name="blue"/>
+      </visual>
+      <xacro:uvc_tube_row name="${name}" side="${side}" i="${i+1}" n="${n}"/>
+    </xacro:if>
+  </xacro:macro>
+  <!-- n row-wise tubes + one collision box, for one side -->
   <xacro:macro name="uvc_lamp_side" params="name side">
-    <xacro:uvc_tube name="${name}_1" y="${side*(panel_y_c - tube_o1)}"/>
-    <xacro:uvc_tube name="${name}_2" y="${side*(panel_y_c - tube_o2)}"/>
-    <xacro:uvc_tube name="${name}_3" y="${side*(panel_y_c + tube_o2)}"/>
-    <xacro:uvc_tube name="${name}_4" y="${side*(panel_y_c + tube_o1)}"/>
+    <xacro:uvc_tube_row name="${name}" side="${side}" i="0" n="${n_tubes}"/>
     <collision name="uvc_lamp_${name}_collision">
       <origin xyz="${panel_x_c} ${side*panel_y_c} ${lamp_z}" rpy="0 0 0"/>
-      <geometry><box size="${panel_len} ${2*tube_o1 + 2*tube_radius} ${2*tube_radius}"/></geometry>
+      <geometry><box size="${panel_len} ${tube_len} ${2*tube_radius}"/></geometry>
     </collision>
   </xacro:macro>
@@ -101,16 +138,48 @@
       <geometry><cylinder radius="${rod_radius}" length="${arm_z - rod_z_bot}"/></geometry>
     </collision>
-    <!-- cross-arm spanning out to both panel centres -->
-    <visual name="uvc_cross_arm">
-      <origin xyz="${rod_x} 0 ${arm_z}" rpy="0 0 0"/>
-      <geometry><box size="${beam_w} ${2*panel_y_c} ${beam_w}"/></geometry>
-      <material name="grey"/>
-    </visual>
-    <collision name="uvc_cross_arm_collision">
-      <origin xyz="${rod_x} 0 ${arm_z}" rpy="0 0 0"/>
-      <geometry><box size="${beam_w} ${2*panel_y_c} ${beam_w}"/></geometry>
+    <!-- horizontal CIRCULAR cross-tube, T-welded to mast top, reaching to each
+         panel's inner edge (cylinder axis along Y -> roll 90 deg) -->
+    <visual name="uvc_cross_tube">
+      <origin xyz="${rod_x} 0 ${arm_z}" rpy="1.5708 0 0"/>
+      <geometry><cylinder radius="${rod_radius}" length="${2*panel_inner}"/></geometry>
+      <material name="grey"/>
+    </visual>
+    <collision name="uvc_cross_tube_collision">
+      <origin xyz="${rod_x} 0 ${arm_z}" rpy="1.5708 0 0"/>
+      <geometry><cylinder radius="${rod_radius}" length="${2*panel_inner}"/></geometry>
     </collision>
     <xacro:uvc_panel name="left"  side="1"/>
     <xacro:uvc_panel name="right" side="-1"/>
+    <!-- weld collars/gussets: a tapered block at each tube-to-panel inner-edge
+         joint, bridging the fat round tube to the thin flat panel -->
+    <xacro:macro name="uvc_weld" params="side">
+      <visual name="uvc_weld_${side}">
+        <origin xyz="${rod_x} ${side*panel_inner} ${arm_z}" rpy="0 0 0"/>
+        <geometry><box size="0.09 0.07 ${2*rod_radius + panel_thick}"/></geometry>
+        <material name="grey"/>
+      </visual>
+      <collision name="uvc_weld_${side}_collision">
+        <origin xyz="${rod_x} ${side*panel_inner} ${arm_z}" rpy="0 0 0"/>
+        <geometry><box size="0.09 0.07 ${2*rod_radius + panel_thick}"/></geometry>
+      </collision>
+    </xacro:macro>
+    <xacro:uvc_weld side="1"/>
+    <xacro:uvc_weld side="-1"/>
+    <!-- camera L-bracket: a forward arm from the panel front edge, then a drop
+         down to the D455 (so the camera hangs forward & below, lens down) -->
+    <xacro:macro name="uvc_cam_bracket" params="side">
+      <visual name="cam_arm_${side}">
+        <origin xyz="${panel_front_x + cam_fwd/2} ${side*panel_y_c} ${arm_z - 0.012}" rpy="0 0 0"/>
+        <geometry><box size="${cam_fwd + 0.02} 0.025 0.02"/></geometry>
+        <material name="grey"/>
+      </visual>
+      <visual name="cam_drop_${side}">
+        <origin xyz="${panel_front_x + cam_fwd} ${side*panel_y_c} ${arm_z - cam_drop/2}" rpy="0 0 0"/>
+        <geometry><box size="0.025 0.025 ${cam_drop}"/></geometry>
+        <material name="grey"/>
+      </visual>
+    </xacro:macro>
+    <xacro:uvc_cam_bracket side="1"/>
+    <xacro:uvc_cam_bracket side="-1"/>
     <inertial>
       <origin xyz="${rod_x} 0 ${arm_z}" rpy="0 0 0"/>
@@ -139,3 +208,40 @@
     <origin xyz="0 0 0" rpy="0 0 0"/>
   </joint>
+  <!-- ── RealSense D455 (real mesh), on the FRONT EDGE of each panel, facing
+       down at the bed. Link frame is pitched +90 so the Gazebo camera sensor's
+       +X axis looks straight down; the mesh is rolled so its lens faces down and
+       its long axis runs across the bed (Y). ── -->
+  <xacro:macro name="uvc_camera" params="name side">
+    <link name="uvc_cam_${name}_link">
+      <visual>
+        <!-- official RealSense d455.stl orientation (rpy pi/2,0,pi/2); link +X
+             points down (joint below), so the lens points down at the bed -->
+        <origin xyz="0 0 0" rpy="1.5708 0 1.5708"/>
+        <geometry>
+          <mesh filename="package://pomona_description/meshes/sensors/d455.stl"
+                scale="${cam_scale} ${cam_scale} ${cam_scale}"/>
+        </geometry>
+        <material name="dark"/>
+      </visual>
+      <collision>
+        <geometry><box size="0.124 0.029 0.026"/></geometry>
+      </collision>
+    </link>
+    <joint name="uvc_cam_${name}_joint" type="fixed">
+      <parent link="base_link"/>
+      <child  link="uvc_cam_${name}_link"/>
+      <!-- panel FRONT edge (+X), over the bed centre (side*panel_y_c), just below
+           the panel; pitched +90 so the sensor looks straight down at the bed -->
+      <origin xyz="${panel_front_x + cam_fwd} ${side*panel_y_c} ${arm_z - cam_drop}" rpy="0 1.5708 0"/>
+    </joint>
+    <!-- REP-103 optical frame (Z forward, X right, Y down) for published images -->
+    <link name="uvc_cam_${name}_optical_frame"/>
+    <joint name="uvc_cam_${name}_optical_joint" type="fixed">
+      <parent link="uvc_cam_${name}_link"/>
+      <child  link="uvc_cam_${name}_optical_frame"/>
+      <origin xyz="0 0 0" rpy="-1.5708 0 -1.5708"/>
+    </joint>
+  </xacro:macro>
+  <xacro:uvc_camera name="left"  side="1"/>
+  <xacro:uvc_camera name="right" side="-1"/>
 </robot>
