Commit message: feat(uvc): render UV-C lamps as per-tube gpu_ray ray-fans
  - UV-C emission is now a per-tube gpu_ray fan firing from each lamp cylinder to
    the ground (15 rays over a +/-15 deg downward arc, range 2.2 m), visualised
    like a lidar scan; lamp tubes glow Gazebo/PurpleGlow.
  - each emitter gets its own link with the pose+roll on the fixed joint (sensor at
    link origin) so URDF->SDF fixed-joint lumping preserves the pose in both the
    xacro and gz-sdf pipelines.
  - drop the old translucent light-curtain / geometry-ray approach and the unused
    uvc_beam material; rslidar viz off so its blue fan doesn't clash.
  - regenerate pomona_gazebo models/pomona_uvc/model.sdf to match.

File: src/pomona_description/urdf/pomona_uvc/urdf/pomona_uvc.urdf (robot description, URDF)
Before this commit: robot pomona, 19 links, 18 joints
Links:
- removed link uvc_beam_link
Joints:
- removed joint uvc_beam_joint

File: src/pomona_description/urdf/pomona_uvc/urdf/pomona_uvc_sim.urdf (robot description, URDF)
Before this commit: robot pomona, 19 links, 18 joints
Links:
- removed link uvc_beam_link
- added link uvc_emit_left_0_link, mass 0.0001
- added link uvc_emit_left_1_link, mass 0.0001
- added link uvc_emit_left_2_link, mass 0.0001
- added link uvc_emit_left_3_link, mass 0.0001
- added link uvc_emit_left_4_link, mass 0.0001
- added link uvc_emit_left_5_link, mass 0.0001
- added link uvc_emit_right_0_link, mass 0.0001
- added link uvc_emit_right_1_link, mass 0.0001
- added link uvc_emit_right_2_link, mass 0.0001
- added link uvc_emit_right_3_link, mass 0.0001
- added link uvc_emit_right_4_link, mass 0.0001
- added link uvc_emit_right_5_link, mass 0.0001
Joints:
- removed joint uvc_beam_joint
- added joint uvc_emit_left_0_joint: type fixed, parent base_link, child uvc_emit_left_0_link, origin xyz=-0.21999999999999997 1.0 0.781 rpy=1.5708 0 0
- added joint uvc_emit_left_1_joint: type fixed, parent base_link, child uvc_emit_left_1_link, origin xyz=-0.10599999999999998 1.0 0.781 rpy=1.5708 0 0
- added joint uvc_emit_left_2_joint: type fixed, parent base_link, child uvc_emit_left_2_link, origin xyz=0.008000000000000007 1.0 0.781 rpy=1.5708 0 0
- added joint uvc_emit_left_3_joint: type fixed, parent base_link, child uvc_emit_left_3_link, origin xyz=0.122 1.0 0.781 rpy=1.5708 0 0
- added joint uvc_emit_left_4_joint: type fixed, parent base_link, child uvc_emit_left_4_link, origin xyz=0.236 1.0 0.781 rpy=1.5708 0 0
- added joint uvc_emit_left_5_joint: type fixed, parent base_link, child uvc_emit_left_5_link, origin xyz=0.35 1.0 0.781 rpy=1.5708 0 0
- added joint uvc_emit_right_0_joint: type fixed, parent base_link, child uvc_emit_right_0_link, origin xyz=-0.21999999999999997 -1.0 0.781 rpy=1.5708 0 0
- added joint uvc_emit_right_1_joint: type fixed, parent base_link, child uvc_emit_right_1_link, origin xyz=-0.10599999999999998 -1.0 0.781 rpy=1.5708 0 0
- added joint uvc_emit_right_2_joint: type fixed, parent base_link, child uvc_emit_right_2_link, origin xyz=0.008000000000000007 -1.0 0.781 rpy=1.5708 0 0
- added joint uvc_emit_right_3_joint: type fixed, parent base_link, child uvc_emit_right_3_link, origin xyz=0.122 -1.0 0.781 rpy=1.5708 0 0
- added joint uvc_emit_right_4_joint: type fixed, parent base_link, child uvc_emit_right_4_link, origin xyz=0.236 -1.0 0.781 rpy=1.5708 0 0
- added joint uvc_emit_right_5_joint: type fixed, parent base_link, child uvc_emit_right_5_link, origin xyz=0.35 -1.0 0.781 rpy=1.5708 0 0

File: src/pomona_description/urdf/pomona_uvc/xacro/common_properties.xacro (robot description, xacro)
@@ -21,8 +21,6 @@
   <material name="orange"><color rgba="1.0 0.424 0.039 1.0"/></material>
   <material name="brown"><color rgba="0.871 0.812 0.765 1.0"/></material>
-  <!-- UV-C lamp "on" violet + translucent projected beam (RViz; Gazebo overrides
-       these with Gazebo/PurpleGlow + Gazebo/DarkMagentaTransparent). -->
+  <!-- UV-C lamp "on" violet (RViz; Gazebo overrides with Gazebo/PurpleGlow). -->
   <material name="uvc_violet"><color rgba="0.60 0.10 0.95 1.0"/></material>
-  <material name="uvc_beam"><color rgba="0.60 0.15 0.95 0.22"/></material>
   <!-- Constants -->
   <xacro:property name="M_PI" value="3.14159"/>

File: src/pomona_description/urdf/pomona_uvc/xacro/gazebo_plugins.xacro (robot description, xacro)
@@ -79,5 +79,8 @@
     <sensor name="rslidar" type="gpu_ray">
       <always_on>true</always_on>
-      <visualize>true</visualize>
+      <!-- viz OFF so the lidar's blue ray fan doesn't clash with the UV-C ray
+           fans (Gazebo Classic hardcodes laser colour → can't recolour either).
+           The lidar still publishes /scan; view it in RViz to recolour it. -->
+      <visualize>false</visualize>
       <update_rate>10</update_rate>
       <ray>
@@ -134,12 +137,81 @@
   </gazebo>
   <!-- ════════════════════════════════════════════════════════════════════
-       UV-C projected beam — translucent violet "light curtain" volume from the
-       lamps down onto the bed. A continuous rendered volume (not discrete rays
-       like the lidar). DarkMagentaTransparent is alpha-blended so the beds show
-       through, tinted violet where the UV-C lands.
-       ════════════════════════════════════════════════════════════════════ -->
-  <gazebo reference="uvc_beam_link">
-    <material>Gazebo/DarkMagentaTransparent</material>
-  </gazebo>
+       UV-C emission — a real Gazebo ray fan per lamp tube (visualised like the
+       lidar laser). Each gpu_ray is posed at its tube, frame rolled +90° so the
+       horizontal scan plane is X-Z (perpendicular to the Y-axis tube). The sweep
+       is a NARROW downward arc (≈120°, centred straight down: −150°..−30°) so it
+       is ONE render camera — NOT a 360° fan, which builds a 6-camera cube-map and
+       (×12 tubes) starved gzserver so the base stopped driving. A thin vertical
+       spread gives the fan some thickness along the tube. Rays terminate on the
+       panel/flaps + bed/plants → real coverage viz. gpu_ray (not ray) per
+       [[gpu-ray-lidar-gotcha]]. NOTE: Classic renders laser rays in fixed
+       blue/turquoise — colour is not configurable (lamps glow PurpleGlow above).
+       Tune samples / update_rate / uvc_ray_count if FPS drops.
+       ════════════════════════════════════════════════════════════════════ -->
+  <xacro:property name="uvc_ray_count" value="${n_tubes}"/>   <!-- gpu_ray sensors per side -->
+  <!-- fire from the lamp tube centreline so the ray origin sits ON the lamp
+       cylinder (the earlier "drop below the flap line" was a workaround for the
+       lumping bug below — no longer needed; downward rays clear the shroud) -->
+  <xacro:property name="emit_z" value="${lamp_z}"/>
+  <!-- CRITICAL: each emitter gets its OWN link, sensor at the link ORIGIN (pose 0).
+       Multiple sensors with <pose> offsets on ONE fixed-jointed link get their pose
+       DROPPED by gazebo's URDF→SDF fixed-joint lumping (verified: all 12 collapsed
+       to base origin, no roll, scanning the wheels at ~0.13 m). Putting the
+       position+roll on the JOINT (like rslidar_link) makes lumping bake it in. -->
+  <xacro:macro name="uvc_ray_emitter" params="name side i n">
+    <xacro:if value="${i &lt; n}">
+      <link name="uvc_emit_${name}_${i}_link">
+        <inertial>
+          <mass value="0.0001"/>
+          <inertia ixx="1e-7" ixy="0" ixz="0" iyy="1e-7" iyz="0" izz="1e-7"/>
+        </inertial>
+      </link>
+      <joint name="uvc_emit_${name}_${i}_joint" type="fixed">
+        <parent link="base_link"/>
+        <child  link="uvc_emit_${name}_${i}_link"/>
+        <origin xyz="${panel_x_c - panel_len/2 + tube_inset_x + i*(panel_len - 2*tube_inset_x)/(n-1)} ${side*panel_y_c} ${emit_z}"
+                rpy="1.5708 0 0"/>
+      </joint>
+      <gazebo reference="uvc_emit_${name}_${i}_link">
+        <sensor name="uvc_emit_${name}_${i}" type="gpu_ray">
+          <pose>0 0 0 0 0 0</pose>
+          <always_on>true</always_on>
+          <visualize>true</visualize>
+          <update_rate>8</update_rate>
+          <ray>
+            <scan>
+              <horizontal>
+                <samples>15</samples>
+                <resolution>1</resolution>
+                <min_angle>-1.8326</min_angle>   <!-- −105° : down-and-back (±15° from straight down, 30° total) -->
+                <max_angle>-1.3090</max_angle>   <!-- −75°  : down-and-fore -->
+              </horizontal>
+              <vertical>
+                <samples>3</samples>
+                <resolution>1</resolution>
+                <min_angle>-0.17</min_angle>
+                <max_angle>0.17</max_angle>
+              </vertical>
+            </scan>
+            <range>
+              <min>0.01</min>
+              <!-- reach the ground: lamp is ~1.02 m AGL straight down; the ±60°
+                   edge rays need ~2 m, so the whole fan lands on the floor (in
+                   crop worlds it terminates earlier on the beds/plants) -->
+              <max>2.2</max>
+              <resolution>0.01</resolution>
+            </range>
+          </ray>
+        </sensor>
+      </gazebo>
+      <xacro:uvc_ray_emitter name="${name}" side="${side}" i="${i+1}" n="${n}"/>
+    </xacro:if>
+  </xacro:macro>
+  <xacro:uvc_ray_emitter name="left"  side="1"  i="0" n="${uvc_ray_count}"/>
+  <xacro:uvc_ray_emitter name="right" side="-1" i="0" n="${uvc_ray_count}"/>
+  <!-- NOTE: these blue ray fans are ALWAYS on. Gazebo Classic keeps a visualised
+       laser sensor alive via the gzclient visual subscription, so SetActive()
+       can't switch them off. The toggleable UV-C signal is the disinfection DOSE
+       map (pomona_uvc → /uvc/dose in RViz), driven by /uvc/* services. -->
   <!-- ════════════════════════════════════════════════════════════════════
        RealSense D455 x2 — one per panel, looking down at each bed

File: src/pomona_description/urdf/pomona_uvc/xacro/uvc_cantilever.xacro (robot description, xacro)
@@ -82,11 +82,11 @@
   <xacro:property name="flap_thick"   value="0.006"/>  <!-- thin shield plate -->
   <xacro:property name="lamp_z" value="${arm_z - panel_thick/2 - tube_radius - 0.004}"/>
-  <!-- UV-C projected beam: a translucent "light curtain" volume from the lamp
-       plane down onto the bed top, so the disinfection looks ON in Gazebo (a
-       continuous rendered violet volume, not discrete rays). Bed top is 0.40 m
-       AGL; base_link sits 0.235 m AGL → bed top = 0.165 in base_link. -->
+  <!-- UV-C emission: rendered by per-tube gpu_ray sensor fans (see
+       gazebo_plugins.xacro) — a downward laser fan out of each lamp tube, like
+       a lidar scan, terminating on the bed/plants. beam_h = lamp-to-bed drop
+       sets the ray range. Bed top is 0.40 m AGL; base_link sits 0.235 m AGL →
+       bed top = 0.165 in base_link. -->
   <xacro:property name="bed_top_z" value="0.165"/>
   <xacro:property name="beam_h"  value="${lamp_z - bed_top_z}"/>
-  <xacro:property name="beam_cz" value="${(lamp_z + bed_top_z)/2.0}"/>
   <!-- housing for one side: flat roof plate + two thin side flaps (skirts) that
        hang down on both long edges so the UV-C only projects onto the bed -->
@@ -215,29 +215,6 @@
     <origin xyz="0 0 0" rpy="0 0 0"/>
   </joint>
-  <!-- ── UV-C beam link: translucent projected "light curtain" under each panel
-       (Gazebo colours it Gazebo/DarkMagentaTransparent). Visual only — no
-       collision (it is light, not a solid). ── -->
-  <link name="uvc_beam_link">
-    <visual name="uvc_beam_left">
-      <origin xyz="${panel_x_c} ${panel_y_c} ${beam_cz}" rpy="0 0 0"/>
-      <geometry><box size="${panel_len*0.95} ${tube_len} ${beam_h}"/></geometry>
-      <material name="uvc_beam"/>
-    </visual>
-    <visual name="uvc_beam_right">
-      <origin xyz="${panel_x_c} ${-panel_y_c} ${beam_cz}" rpy="0 0 0"/>
-      <geometry><box size="${panel_len*0.95} ${tube_len} ${beam_h}"/></geometry>
-      <material name="uvc_beam"/>
-    </visual>
-    <inertial>
-      <origin xyz="${panel_x_c} 0 ${beam_cz}" rpy="0 0 0"/>
-      <mass value="0.001"/>
-      <inertia ixx="1e-6" ixy="0" ixz="0" iyy="1e-6" iyz="0" izz="1e-6"/>
-    </inertial>
-  </link>
-  <joint name="uvc_beam_joint" type="fixed">
-    <parent link="base_link"/>
-    <child  link="uvc_beam_link"/>
-    <origin xyz="0 0 0" rpy="0 0 0"/>
-  </joint>
+  <!-- UV-C emission is rendered by gpu_ray sensors on uvc_lamps_link
+       (gazebo_plugins.xacro) — a downward laser fan per lamp tube. -->
   <!-- ── RealSense D455 (real mesh), on the FRONT EDGE of each panel, facing
        down at the bed. Link frame is pitched +90 so the Gazebo camera sensor's
